File: pcb/init.brd (EAGLE design)
At the start: 53 x 20.3 mm, 6 parts

Commit message: pcb
Parts:
- moved JP6 8.89 mm to (20.3, 6.35)
- moved JP5 7.62 mm to (12.7, 14.0)
Connections:
- removed net N$6: JP5.2, SENSOR.2
- new net 5V: JP6.4, SENSOR.1
- new net N$1: JP5.1, SENSOR.2
- new net N$2: COOLER.2, JP6.3
- net GND: now also JP5.2; no longer JP5.4, TERMO.2
- net N$5: now also JP5.4, TERMO.2; no longer COOLER.2, JP6.4
- net VCC: no longer JP5.1, JP6.3, SENSOR.1
Routing:
- net VCC: track 85.3 -> 17.8 mm
- net N$1: track 0.00 -> 28.9 mm
- net 5V: track 0.00 -> 19.6 mm
- net N$6: track 18.8 -> 0.00 mm
- net N$2: track 0.00 -> 18.8 mm
- net GND: track 17.8 -> 29.6 mm
- net N$5: track 28.8 -> 17.8 mm
- net N$9: track 19.1 -> 10.2 mm
- net N$3: track 10.2 -> 18.4 mm
Other:
- board size 53 x 20.3 mm -> 55 x 20 mm
